Commit message: changes in documentation, new maps folder, and fixbugs

File: Robots/Robot1/R1_urdf/Robot_Linz.urdf (robot description, URDF)
Before this commit: robot flexible, 9 links, 8 joints
Links:
- link PLS200: geometry visual mesh filename=package://R1_urdf/bot_PLS200.dae scale=0.025 0.025 0.025
- link base_link: geometry visual mesh filename=package://R1_urdf/bot_body.dae scale=0.025 0.025 0.025
- link kinect_rgb: geometry visual mesh filename=package://R1_urdf/bot_kinect.dae scale=0.025 0.025 0.025
- link wheel_1: geometry visual mesh filename=package://R1_urdf/bot_wheel.dae scale=0.025 0.025 0.025
- link wheel_2: geometry visual mesh filename=package://R1_urdf/bot_wheel.dae scale=0.025 0.025 0.025
- link wheel_3: geometry visual mesh filename=package://R1_urdf/bot_wheel.dae scale=0.025 0.025 0.025
- link wheel_4: geometry visual mesh filename=package://R1_urdf/bot_wheel.dae scale=0.025 0.025 0.025

Commit message: cleaning code, fix bug of server, problem with mutex

File: Robots/Robot1/R1_urdf/Robot_Linz.urdf (robot description, URDF)
Before this commit: robot flexible, 9 links, 8 joints
Links:
- added link odom
Joints:
- added joint odom_base: type continuous, parent odom, child base_link

Commit message: navigation stack ok

File: Robots/Robot1/R1_urdf/Robot_Linz.urdf (robot description, URDF)
Before this commit: robot flexible, 10 links, 9 joints
Links:
- removed link head
- removed link medida
- removed link odom
Joints:
- removed joint head_swivel
- removed joint odom_base
- removed joint tobox3
- joint tobox2: parent head -> base_link
- joint tobox5: parent head -> base_link
- joint tobox6: parent head -> base_link
- joint tobox7: parent head -> base_link
- joint tobox8: parent head -> base_link
- joint tobox9: parent head -> base_link

Commit message: scheme for power supply for sensor, doc in word

File: Robots/Robot1/R1_urdf/Robot_Linz.urdf (robot description, URDF)
Before this commit: robot flexible, 7 links, 6 joints
Joints:
- removed joint tobox2
- removed joint tobox5
- removed joint tobox6
- removed joint tobox7
- removed joint tobox8
- removed joint tobox9
- added joint join_1: type continuous, parent base_link, child wheel_1, origin xyz=0.235 -0.17 0 rpy=0 0 0, axis 0 0 1
- added joint join_2: type continuous, parent base_link, child wheel_2, origin xyz=0.235 0.17 0 rpy=0 0 3.14, axis 0 0 1
- added joint join_3: type continuous, parent base_link, child wheel_3, origin xyz=-0.235 -0.17 0 rpy=0 0 0 , axis 0 0 1
- added joint join_4: type continuous, parent base_link, child wheel_4, origin xyz=-0.235 0.17 0 rpy=0 0 3.14, axis 0 0 1
- added joint join_5: type continuous, parent base_link, child kinect_rgb, origin xyz=0.320 0 0.555 rpy=-1.57 0 -1.570
- added joint join_6: type continuous, parent base_link, child PLS200, origin xyz=0.420 0 0.26 rpy=0 0 0
